Commit message: fixed xacro model

File: urdf/robot.urdf.xacro (robot description, xacro)
@@ -30,5 +30,5 @@
     <inertial>
       <origin xyz="0 0 0" rpy="0 0 0"/>
-      <mass value="{mass_base}"/>
+      <mass value="${mass_base}"/>
       <inertia
         ixx="0.0208"
@@ -87,4 +87,24 @@
   </joint>
   </xacro:macro>
+  <!-- Support wheel -->
+  <xacro:macro name="support_wheel" params="name x y z">
+  <link name="${name}">
+    <visual>
+      <geometry>
+        <sphere radius="0.03"/>
+      </geometry>
+    </visual>
+    <collision>
+      <geometry>
+        <sphere radius="0.03"/>
+      </geometry>
+    </collision>
+  </link>
+  <joint name="${name}_joint" type="fixed">
+    <parent link="base_link"/>
+    <child link="${name}"/>
+    <origin  xyz="${x} ${y} ${z}" rpy="0 0 0"/>
+  </joint>
+  </xacro:macro>
   <!-- Sensors -->
   <xacro:range_sensor_mount name="range_front" x="0.21" y="0.0" z="0.05" roll="0" pitch="0" yaw="0"/>
@@ -94,4 +114,6 @@
   <xacro:wheel name="left_wheel" y_offset="${wheel_y_offset}"/>
   <xacro:wheel name="right_wheel" y_offset="-${wheel_y_offset}"/>
+  <xacro:support_wheel name="front_support_wheel" x="${wheel_y_offset/2}" y="0" z="${- base_height/2 + wheel_radius/2}"/>
+  <xacro:support_wheel name="back_support_wheel" x="${- wheel_y_offset/2}" y="0" z="${- base_height/2 + wheel_radius/2}"/>
   <gazebo>
     <plugin

Commit message: add laser scans and some bug fixed

File: urdf/robot.urdf.xacro (robot description, xacro)
@@ -72,5 +72,5 @@
     </joint>
   </xacro:macro>
-  <xacro:macro name="range_sensor_mount" params="name x y z roll pitch yaw">
+  <xacro:macro name="range_sensor_mount" params="name x y z roll pitch yaw topic_name">
   <link name="${name}">
     <visual>
@@ -80,4 +80,16 @@
       <material name="robot_blue"/>
     </visual>
+    <collision>
+      <geometry>
+        <box size="0.02 0.02 0.02"/>
+      </geometry>
+    </collision>
+    <inertial>
+      <mass value="0.01"/>
+      <inertia
+        ixx="1e-6" ixy="0" ixz="0"
+        iyy="1e-6" iyz="0"
+        izz="1e-6"/>
+    </inertial>
   </link>
   <joint name="${name}_joint" type="fixed">
@@ -86,29 +98,39 @@
     <origin xyz="${x} ${y} ${z}" rpy="${roll} ${pitch} ${yaw}"/>
   </joint>
-  </xacro:macro>
-  <!-- Support wheel -->
+</xacro:macro>
   <xacro:macro name="support_wheel" params="name x y z">
-  <link name="${name}">
-    <visual>
-      <geometry>
-        <sphere radius="0.03"/>
-      </geometry>
-    </visual>
-    <collision>
-      <geometry>
-        <sphere radius="0.03"/>
-      </geometry>
-    </collision>
-  </link>
-  <joint name="${name}_joint" type="fixed">
-    <parent link="base_link"/>
-    <child link="${name}"/>
-    <origin  xyz="${x} ${y} ${z}" rpy="0 0 0"/>
-  </joint>
+    <link name="${name}">
+      <visual>
+        <geometry>
+          <sphere radius="0.03"/>
+        </geometry>
+        <material name="robot_gray"/>
+      </visual>
+      <collision>
+        <geometry>
+          <sphere radius="0.03"/>
+        </geometry>
+      </collision>
+      <inertial>
+        <mass value="0.05"/>
+        <inertia
+          ixx="1e-5"
+          ixy="0.0"
+          ixz="0.0"
+          iyy="1e-5"
+          iyz="0.0"
+          izz="1e-5"/>
+      </inertial>
+    </link>
+    <joint name="${name}_joint" type="fixed">
+      <parent link="base_link"/>
+      <child link="${name}"/>
+      <origin xyz="${x} ${y} ${z}" rpy="0 0 0"/>
+    </joint>
   </xacro:macro>
   <!-- Sensors -->
-  <xacro:range_sensor_mount name="range_front" x="0.21" y="0.0" z="0.05" roll="0" pitch="0" yaw="0"/>
-  <xacro:range_sensor_mount name="range_left"  x="0.00" y="0.21" z="0.05" roll="0" pitch="0" yaw="1.5708"/>
-  <xacro:range_sensor_mount name="range_right" x="0.00" y="-0.21" z="0.05" roll="0" pitch="0" yaw="-1.5708"/>
+  <xacro:range_sensor_mount name="range_front" x="0.21" y="0.0" z="0.05" roll="0" pitch="0" yaw="0" topic_name="/range_front_raw"/>
+  <xacro:range_sensor_mount name="range_left"  x="0.00" y="0.21" z="0.05" roll="0" pitch="0" yaw="1.5708" topic_name="/range_left_raw"/>
+  <xacro:range_sensor_mount name="range_right" x="0.00" y="-0.21" z="0.05" roll="0" pitch="0" yaw="-1.5708" topic_name="/range_right_raw"/>
   <!-- Колёса -->
   <xacro:wheel name="left_wheel" y_offset="${wheel_y_offset}"/>
@@ -142,5 +164,5 @@
       filename="gz-sim-joint-state-publisher-system"
       name="gz::sim::systems::JointStatePublisher">
-      <topic>/world/empty/model/diff_drive/joint_state</topic>
+      <topic>/world/Depot/model/diff_drive/joint_state</topic>
     </plugin>
     <plugin
@@ -153,3 +175,75 @@
     </plugin>
   </gazebo>
+  <gazebo reference="range_front">
+    <sensor name="range_front_sensor" type="gpu_lidar">
+      <always_on>true</always_on>
+      <visualize>true</visualize>
+      <update_rate>10</update_rate>
+      <topic>range_front</topic>
+      <lidar>
+        <scan>
+          <horizontal>
+            <samples>1</samples>
+            <resolution>1</resolution>
+            <min_angle>0.0</min_angle>
+            <max_angle>0.0</max_angle>
+          </horizontal>
+        </scan>
+        <range>
+          <min>0.05</min>
+          <max>5.0</max>
+          <resolution>0.01</resolution>
+        </range>
+      </lidar>
+      <plugin name="dummy" filename="dummyfile"/>
+    </sensor>
+  </gazebo>
+  <gazebo reference="range_left">
+    <sensor name="range_left_sensor" type="gpu_lidar">
+      <always_on>true</always_on>
+      <visualize>true</visualize>
+      <update_rate>10</update_rate>
+      <topic>range_left</topic>
+      <lidar>
+        <scan>
+          <horizontal>
+            <samples>1</samples>
+            <resolution>1</resolution>
+            <min_angle>0.0</min_angle>
+            <max_angle>0.0</max_angle>
+          </horizontal>
+        </scan>
+        <range>
+          <min>0.05</min>
+          <max>5.0</max>
+          <resolution>0.01</resolution>
+        </range>
+      </lidar>
+      <plugin name="dummy" filename="dummyfile"/>
+    </sensor>
+  </gazebo>
+  <gazebo reference="range_right">
+    <sensor name="range_right_sensor" type="gpu_lidar">
+      <always_on>true</always_on>
+      <visualize>true</visualize>
+      <update_rate>10</update_rate>
+      <topic>range_right</topic>
+      <lidar>
+        <scan>
+          <horizontal>
+            <samples>1</samples>
+            <resolution>1</resolution>
+            <min_angle>0.0</min_angle>
+            <max_angle>0.0</max_angle>
+          </horizontal>
+        </scan>
+        <range>
+          <min>0.05</min>
+          <max>5.0</max>
+          <resolution>0.01</resolution>
+        </range>
+      </lidar>
+      <plugin name="dummy" filename="dummyfile"/>
+    </sensor>
+  </gazebo>
 </robot>

Commit message: added node to fixes range sensors frame id, added lidar to make costmap

File: urdf/robot.urdf.xacro (robot description, xacro)
@@ -40,4 +40,11 @@
     </inertial>
   </link>
+  <link name="base_footprint">
+  </link>
+  <joint name="base_joint" type="fixed">
+    <parent link="base_link"/>
+    <child link="base_footprint"/>
+    <origin xyz="0.0 0.0 ${-(base_height/2 + wheel_radius/2)}" rpy="0 0 0"/>
+  </joint>
   <!-- Макрос колеса -->
   <xacro:macro name="wheel" params="name y_offset">
@@ -147,8 +154,8 @@
       <wheel_radius>0.03</wheel_radius>
       <odom_publish_frequency>50</odom_publish_frequency>
-      <topic>model/diff_drive/cmd_vel</topic>
+      <topic>/cmd_vel</topic>
       <odom_topic>model/diff_drive/odometry</odom_topic>
       <tf_topic>model/diff_drive/pose</tf_topic>
-      <frame_id>diff_drive/odom</frame_id>
+      <frame_id>odom</frame_id>
       <child_frame_id>base_link</child_frame_id>
       <min_linear_velocity>-1.0</min_linear_velocity>
@@ -247,3 +254,55 @@
     </sensor>
   </gazebo>
+  <xacro:macro name="lidar_sensor_mount" params="name x y z roll pitch yaw ">
+    <link name="${name}">
+      <visual>
+        <geometry>
+          <box size="0.02 0.02 0.02"/>
+        </geometry>
+        <material name="robot_blue"/>
+      </visual>
+      <collision>
+        <geometry>
+          <box size="0.02 0.02 0.02"/>
+        </geometry>
+      </collision>
+      <inertial>
+        <mass value="0.01"/>
+        <inertia
+          ixx="1e-6" ixy="0" ixz="0"
+          iyy="1e-6" iyz="0"
+          izz="1e-6"/>
+      </inertial>
+    </link>
+    <joint name="${name}_joint" type="fixed">
+      <parent link="base_link"/>
+      <child link="${name}"/>
+      <origin xyz="${x} ${y} ${z}" rpy="${roll} ${pitch} ${yaw}"/>
+    </joint>
+  </xacro:macro>
+  <xacro:lidar_sensor_mount name="lidar_sensor" x="0.00" y="-0.21" z="${base_height/2 + 0.01}" roll="0" pitch="0" yaw="0"/>
+  <gazebo reference="lidar_sensor">
+    <sensor name="range_lidar_sensor" type="gpu_lidar">
+      <always_on>true</always_on>
+      <visualize>true</visualize>
+      <update_rate>10</update_rate>
+      <topic>range_lidar</topic>
+      <lidar>
+        <scan>
+          <horizontal>
+            <samples>360</samples>
+            <resolution>1</resolution>
+            <min_angle>0</min_angle>
+            <max_angle>6.28</max_angle>
+          </horizontal>
+        </scan>
+        <range>
+          <min>0.05</min>
+          <max>5.0</max>
+          <resolution>0.01</resolution>
+        </range>
+      </lidar>
+      <plugin name="dummy" filename="dummyfile"/>
+    </sensor>
+  </gazebo>
 </robot>
